File: MDBT40-Wing.sch (KiCad schematic (older format))
At the start: 3 parts, among them J1 Left, J2 Right, U1 MDBT40

Commit message: Final touches
Other:
- note added: "Designed by K.T.E.C."
Changed lines of the file:
@@
 LIBS:valves
 LIBS:mdbt40
+LIBS:ktec_logo
+LIBS:MDBT40-Wing-cache
 EELAYER 25 0
 EELAYER END
@@
 Comment4 ""
 $EndDescr
-$Comp
-L MDBT40 U1
-U 1 1 58DA2DAB
-P 4900 3550
-F 0 "U1" H 4900 4500 60  0000 C CNN
-F 1 "MDBT40" H 4900 3550 60  0000 C CNN
-F 2 "mdbt40_carrier:MDBT40-Carrier" H 5250 3800 60  0001 C CNN
-F 3 "" H 5250 3800 60  0001 C CNN
-	1    4900 3550
-	1    0    0    -1
-$EndComp
 $Comp
 L CONN_01X21 J1
@@
 Wire Bus Line
 	3100 2750 3100 4850
+$Comp
+L MDBT40 U1
+U 1 1 58DAF3A7
+P 4900 3550
+F 0 "U1" H 4900 4500 60  0000 C CNN
+F 1 "MDBT40" H 4900 3550 60  0000 C CNN
+F 2 "mdbt40_carrier:MDBT40-Carrier" H 5250 3800 60  0001 C CNN
+F 3 "" H 5250 3800 60  0001 C CNN
+	1    4900 3550
+	1    0    0    -1
+$EndComp
+$Comp
+L LOGO #G1
+U 1 1 58DAF75E
+P 7700 5500
+F 0 "#G1" H 7700 5177 60  0001 C CNN
+F 1 "LOGO" H 7700 5823 60  0001 C CNN
+F 2 "ktec_logo:ktec_logo" H 7700 5500 60  0001 C CNN
+F 3 "" H 7700 5500 60  0001 C CNN
+	1    7700 5500
+	1    0    0    -1
+$EndComp
+Text Notes 7950 5750 0    60   ~ 0
+Designed by K.T.E.C.
 $EndSCHEMATC

Commit message: update design
Parts:
- removed J1: Left, Pin_Headers:Pin_Header_Straight_1x21_Pitch1.27mm, symbol CONN_01X21
- removed J2: Right, Pin_Headers:Pin_Header_Straight_1x21_Pitch1.27mm, symbol CONN_01X21
- added J1: LEFT, Pin_Headers:Pin_Header_Straight_1x13_Pitch2.54mm, symbol CONN_01X13
- added J2: RIGHT, Pin_Headers:Pin_Header_Straight_1x13_Pitch2.54mm, symbol CONN_01X13
- added J3: BOTTOM, Pin_Headers:Pin_Header_Straight_1x10_Pitch2.54mm, symbol CONN_01X10
- added J4: DCC, SMD_Packages:1Pin, symbol CONN_01X01
- added J5: DEC2, SMD_Packages:1Pin, symbol CONN_01X01
- added JP1: Jumper, Connectors:GS2, symbol Jumper
Connections:
- net 13 is gone; now on net GND: U1.13 (GND)
- net 2 is gone; now on net GND: U1.2 (GND)
- net 25 is gone; now on net GND: U1.25 (GND)
- net 42 is gone; now on net GND: U1.42 (GND)
- net 1 renamed GND
- net GND: now also J1.1 (P1)
- net 10 renamed P0.27
- net P0.27: now also J1.9 (P9)
- net 11 renamed P0.28
- net P0.28: now also J1.10 (P10)
- net 12 renamed P0.29
- net P0.29: now also J1.11 (P11)
- net 14 renamed VDD
- net VDD: now also J1.13 (P13), JP1.2
- net 15 renamed DCC
- net DCC: now also J4.1 (P1)
- net 16 renamed P0.30
- net P0.30: now also J1.12 (P12)
- net 17 renamed P0.00
- net P0.00: now also J3.1 (P1)
- net 18 renamed P0.01
- net P0.01: now also J3.2 (P2)
- net 19 renamed P0.02
- net P0.02: now also J3.3 (P3)
- net 20 renamed P0.03
- net P0.03: now also J3.4 (P4)
- net 21 renamed P0.04
- net P0.04: now also J3.5 (P5)
- net 22 renamed P0.05
- net P0.05: now also J3.6 (P6)
- net 23 renamed P0.06
- net P0.06: now also J3.7 (P7)
- net 24 renamed P0.07
- net P0.07: now also J3.8 (P8)
- net 26 renamed P0.08
- net P0.08: now also J2.13 (P13)
- net 27 renamed P0.09
- net P0.09: now also J2.12 (P12)
- net 28 renamed P0.10
- net P0.10: now also J2.11 (P11)
- net 29 renamed P0.11
- net P0.11: now also J2.10 (P10)
- net 3 renamed AVDD
- net AVDD: now also J1.2 (P2), JP1.1
- net 30 renamed P0.12
- net P0.12: now also J2.9 (P9)
- net 31 renamed P0.13
- net P0.13: now also J2.8 (P8)
- net 32 renamed P0.14
- net P0.14: now also J2.7 (P7)
- net 33 renamed P0.15
- net P0.15: now also J2.6 (P6)
- net 34 renamed P0.16
- net P0.16: now also J2.5 (P5)
- net 35 renamed SWDIO
- net SWDIO: now also J3.9 (P9)
- net 36 renamed SWCLK
- net SWCLK: now also J3.10 (P10)
- net 37 renamed P0.17
- net P0.17: now also J2.4 (P4)
- net 38 renamed P0.18
- net P0.18: now also J2.3 (P3)
- net 39 renamed P0.19
- net P0.19: now also J2.2 (P2)
- net 4 renamed P0.21
- net P0.21: now also J1.3 (P3)
- net 40 renamed P0.20
- net P0.20: now also J2.1 (P1)
- net 41 renamed DEC2
- net DEC2: now also J5.1 (P1)
- net 5 renamed P0.22
- net P0.22: now also J1.4 (P4)
- net 6 renamed P0.23
- net P0.23: now also J1.5 (P5)
- net 7 renamed P0.24
- net P0.24: now also J1.6 (P6)
- net 8 renamed P0.25
- net P0.25: now also J1.7 (P7)
- net 9 renamed P0.26
- net P0.26: now also J1.8 (P8)

Commit message: Design #6
Parts:
- removed J1: LEFT, Pin_Headers:Pin_Header_Straight_1x13_Pitch2.54mm, symbol CONN_01X13
- removed J2: RIGHT, Pin_Headers:Pin_Header_Straight_1x13_Pitch2.54mm, symbol CONN_01X13
- removed J3: BOTTOM, Pin_Headers:Pin_Header_Straight_1x10_Pitch2.54mm, symbol CONN_01X10
- added J1: LEFT, Pin_Headers:Pin_Header_Straight_1x14_Pitch2.54mm, symbol CONN_01X14
- added J2: RIGHT, Pin_Headers:Pin_Header_Straight_1x14_Pitch2.54mm, symbol CONN_01X14
- added J3: BOTTOM, Pin_Headers:Pin_Header_Straight_1x08_Pitch2.54mm, symbol CONN_01X08
Connections:
- net AVDD: now also J1.2 (P2)
- net GND: now also J1.1 (P1)
- net P0.00: now also J3.1 (P1)
- net P0.01: now also J3.2 (P2)
- net P0.02: now also J3.3 (P3)
- net P0.03: now also J3.4 (P4)
- net P0.04: now also J3.5 (P5)
- net P0.05: now also J3.6 (P6)
- net P0.06: now also J3.7 (P7)
- net P0.07: now also J3.8 (P8)
- net P0.08: now also J2.13 (P13)
- net P0.09: now also J2.12 (P12)
- net P0.10: now also J2.11 (P11)
- net P0.11: now also J2.10 (P10)
- net P0.12: now also J2.9 (P9)
- net P0.13: now also J2.8 (P8)
- net P0.14: now also J2.7 (P7)
- net P0.15: now also J2.6 (P6)
- net P0.16: now also J2.5 (P5)
- net P0.17: now also J2.4 (P4)
- net P0.18: now also J2.3 (P3)
- net P0.19: now also J2.2 (P2)
- net P0.20: now also J2.1 (P1)
- net P0.21: now also J1.3 (P3)
- net P0.22: now also J1.4 (P4)
- net P0.23: now also J1.5 (P5)
- net P0.24: now also J1.6 (P6)
- net P0.25: now also J1.7 (P7)
- net P0.26: now also J1.8 (P8)
- net P0.27: now also J1.9 (P9)
- net P0.28: now also J1.10 (P10)
- net P0.29: now also J1.11 (P11)
- net P0.30: now also J1.12 (P12)
- net SWCLK: now also J1.14 (P14)
- net SWDIO: now also J2.14 (P14)
- net VDD: now also J1.13 (P13)
Changed lines of the file:
@@
 Text Notes 7950 5750 0    60   ~ 0
 Designed by K.T.E.C.
-$Comp
-L CONN_01X13 J1
-U 1 1 58DBF131
-P 2550 3350
-F 0 "J1" H 2550 4050 50  0000 C CNN
-F 1 "LEFT" V 2650 3350 50  0000 C CNN
-F 2 "Pin_Headers:Pin_Header_Straight_1x13_Pitch2.54mm" H 2550 3350 50  0001 C CNN
-F 3 "" H 2550 3350 50  0001 C CNN
-	1    2550 3350
-	-1   0    0    -1
-$EndComp
 Entry Wire Line
 	3000 2750 3100 2850
@@
 Text Label 2750 3950 0    60   ~ 0
 VDD
-$Comp
-L CONN_01X13 J2
-U 1 1 58DC035C
-P 7150 3350
-F 0 "J2" H 7150 4050 50  0000 C CNN
-F 1 "RIGHT" V 7250 3350 50  0000 C CNN
-F 2 "Pin_Headers:Pin_Header_Straight_1x13_Pitch2.54mm" H 7150 3350 50  0001 C CNN
-F 3 "" H 7150 3350 50  0001 C CNN
-	1    7150 3350
-	1    0    0    -1
-$EndComp
 Entry Wire Line
 	6600 2850 6700 2750
@@
 Entry Wire Line
 	6600 4050 6700 3950
-$Comp
-L CONN_01X10 J3
-U 1 1 58DC0DEE
-P 2550 4700
-F 0 "J3" H 2550 5250 50  0000 C CNN
-F 1 "BOTTOM" V 2650 4700 50  0000 C CNN
-F 2 "Pin_Headers:Pin_Header_Straight_1x10_Pitch2.54mm" H 2550 4700 50  0001 C CNN
-F 3 "" H 2550 4700 50  0001 C CNN
-	1    2550 4700
-	-1   0    0    -1
-$EndComp
 Wire Bus Line
 	3500 5200 6200 5200
@@
 Text Label 6700 3950 0    60   ~ 0
 P0.08
-Wire Wire Line
-	2750 4250 3000 4250
-Entry Wire Line
-	3000 4250 3100 4350
+Entry Wire Line
+	3000 4050 3100 4150
 Entry Wire Line
 	3000 4350 3100 4450
@@
 Entry Wire Line
 	3000 5050 3100 5150
-Entry Wire Line
-	3000 5150 3100 5250
 Wire Wire Line
 	2750 4350 3000 4350
@@
 Wire Wire Line
 	2750 5050 3000 5050
-Wire Wire Line
-	3000 5150 2750 5150
-Text Label 2750 4250 0    60   ~ 0
+Text Label 2750 4350 0    60   ~ 0
 P0.00
-Text Label 2750 4350 0    60   ~ 0
+Text Label 2750 4450 0    60   ~ 0
 P0.01
-Text Label 2750 4450 0    60   ~ 0
+Text Label 2750 4550 0    60   ~ 0
 P0.02
-Text Label 2750 4550 0    60   ~ 0
+Text Label 2750 4650 0    60   ~ 0
 P0.03
-Text Label 2750 4650 0    60   ~ 0
+Text Label 2750 4750 0    60   ~ 0
 P0.04
-Text Label 2750 4750 0    60   ~ 0
+Text Label 2750 4850 0    60   ~ 0
 P0.05
-Text Label 2750 4850 0    60   ~ 0
+Text Label 2750 4950 0    60   ~ 0
 P0.06
-Text Label 2750 4950 0    60   ~ 0
+Text Label 2750 5050 0    60   ~ 0
 P0.07
-Text Label 2750 5150 0    60   ~ 0
+Text Label 2750 4050 0    60   ~ 0
 SWCLK
-Text Label 2750 5050 0    60   ~ 0
+Text Label 6700 4050 0    60   ~ 0
 SWDIO
 Wire Wire Line
@@
 Text Label 6700 4400 0    60   ~ 0
 DCC
+$Comp
+L CONN_01X14 J1
+U 1 1 58DDBC41
+P 2550 3400
+F 0 "J1" H 2550 4150 50  0000 C CNN
+F 1 "LEFT" V 2650 3400 50  0000 C CNN
+F 2 "Pin_Headers:Pin_Header_Straight_1x14_Pitch2.54mm" H 2550 3400 50  0001 C CNN
+F 3 "" H 2550 3400 50  0001 C CNN
+	1    2550 3400
+	-1   0    0    -1
+$EndComp
+Wire Wire Line
+	2750 4050 3000 4050
+$Comp
+L CONN_01X14 J2
+U 1 1 58DDC122
+P 7150 3400
+F 0 "J2" H 7150 4150 50  0000 C CNN
+F 1 "RIGHT" V 7250 3400 50  0000 C CNN
+F 2 "Pin_Headers:Pin_Header_Straight_1x14_Pitch2.54mm" H 7150 3400 50  0001 C CNN
+F 3 "" H 7150 3400 50  0001 C CNN
+	1    7150 3400
+	1    0    0    -1
+$EndComp
+Entry Wire Line
+	6600 4150 6700 4050
+Wire Wire Line
+	6700 4050 6950 4050
+$Comp
+L CONN_01X08 J3
+U 1 1 58DDC5B6
+P 2550 4700
+F 0 "J3" H 2550 5150 50  0000 C CNN
+F 1 "BOTTOM" V 2650 4700 50  0000 C CNN
+F 2 "Pin_Headers:Pin_Header_Straight_1x08_Pitch2.54mm" H 2550 4700 50  0001 C CNN
+F 3 "" H 2550 4700 50  0001 C CNN
+	1    2550 4700
+	-1   0    0    -1
+$EndComp
 $EndSCHEMATC

Commit message: Design #7
Parts:
- J3: symbol CONN_01X08 -> CONN_02X04
Other:
- moved on the sheet: J3
Changed lines of the file:
@@
 	3500 2750 3100 2750
 Wire Bus Line
-	3100 2750 3100 5300
+	3100 2750 3100 5200
 Wire Wire Line
 	2750 2750 3000 2750
@@
 	3000 4050 3100 4150
 Entry Wire Line
-	3000 4350 3100 4450
-Entry Wire Line
 	3000 4450 3100 4550
 Entry Wire Line
@@
 Entry Wire Line
 	3000 4750 3100 4850
-Entry Wire Line
-	3000 4850 3100 4950
-Entry Wire Line
-	3000 4950 3100 5050
-Entry Wire Line
-	3000 5050 3100 5150
-Wire Wire Line
-	2750 4350 3000 4350
-Wire Wire Line
-	3000 4450 2750 4450
+Wire Wire Line
+	2750 4450 3000 4450
 Wire Wire Line
 	3000 4550 2750 4550
 Wire Wire Line
-	2750 4650 3000 4650
-Wire Wire Line
-	3000 4750 2750 4750
-Wire Wire Line
-	2750 4850 3000 4850
-Wire Wire Line
-	3000 4950 2750 4950
-Wire Wire Line
-	2750 5050 3000 5050
-Text Label 2750 4350 0    60   ~ 0
+	3000 4650 2750 4650
+Wire Wire Line
+	2750 4750 3000 4750
+Text Label 2750 4450 0    60   ~ 0
 P0.00
-Text Label 2750 4450 0    60   ~ 0
-P0.01
 Text Label 2750 4550 0    60   ~ 0
 P0.02
 Text Label 2750 4650 0    60   ~ 0
-P0.03
+P0.04
 Text Label 2750 4750 0    60   ~ 0
-P0.04
-Text Label 2750 4850 0    60   ~ 0
-P0.05
-Text Label 2750 4950 0    60   ~ 0
 P0.06
-Text Label 2750 5050 0    60   ~ 0
-P0.07
 Text Label 2750 4050 0    60   ~ 0
 SWCLK
@@
 	6700 4050 6950 4050
 $Comp
-L CONN_01X08 J3
+L CONN_02X04 J3
 U 1 1 58DDC5B6
-P 2550 4700
-F 0 "J3" H 2550 5150 50  0000 C CNN
-F 1 "BOTTOM" V 2650 4700 50  0000 C CNN
-F 2 "Pin_Headers:Pin_Header_Straight_1x08_Pitch2.54mm" H 2550 4700 50  0001 C CNN
-F 3 "" H 2550 4700 50  0001 C CNN
-	1    2550 4700
+P 2500 4600
+F 0 "J3" H 2500 4850 50  0000 C CNN
+F 1 "BOTTOM" V 2600 4600 50  0000 C CNN
+F 2 "Pin_Headers:Pin_Header_Straight_1x08_Pitch2.54mm" H 2500 4600 50  0001 C CNN
+F 3 "" H 2500 4600 50  0001 C CNN
+	1    2500 4600
 	-1   0    0    -1
 $EndComp
+Wire Bus Line
+	3100 5200 1900 5200
+Wire Bus Line
+	1900 5200 1900 4200
+Entry Wire Line
+	1900 4550 2000 4450
+Entry Wire Line
+	1900 4650 2000 4550
+Entry Wire Line
+	1900 4750 2000 4650
+Entry Wire Line
+	1900 4850 2000 4750
+Wire Wire Line
+	2250 4450 2000 4450
+Wire Wire Line
+	2250 4550 2000 4550
+Wire Wire Line
+	2250 4650 2000 4650
+Wire Wire Line
+	2250 4750 2000 4750
+Text Label 2000 4450 0    60   ~ 0
+P0.01
+Text Label 2000 4550 0    60   ~ 0
+P0.03
+Text Label 2000 4650 0    60   ~ 0
+P0.05
+Text Label 2000 4750 0    60   ~ 0
+P0.07
 $EndSCHEMATC
